Commit message: Oppgave 2 - refined

File: src/qube_description/urdf/qube.macro.xacro (robot description, xacro)
@@ -1,11 +1,63 @@
 <?xml version="1.0"?>
-<robot xmlns:xacro="http://www.ros.org/wiki/xacro" name="qube">
-  <xacro:include filename="$(find qube_description)/urdf/qube.urdf.xacro"/>
-  <link name="world"/>
-  <xacro:qube prefix=""/>
-  <joint name="world_joint" type="fixed">       <!-- plasser Quben i origo -->
-    <parent link="world"/>
-    <child link="base_link"/>
-    <origin xyz="0 0 0" rpy="0 0 0"/>
-  </joint>
+<robot xmlns:xacro="http://www.ros.org/wiki/xacro">
+  <!-- Mål på delene i meter -->
+  <xacro:property name="stator_size"       value="0.102" />   <!-- svart boks -->
+  <xacro:property name="rotor_radius"      value="0.025" />   <!-- disk radius -->
+  <xacro:property name="rotor_length"      value="0.01"  />   <!-- disk tykkelse -->
+  <xacro:property name="indicator_length"  value="0.025" />   <!-- viser lengde -->
+  <xacro:property name="indicator_width"   value="0.005" />   <!-- viser bredde -->
+  <!-- prefix-parameteren gjør at makroen kan brukes flere ganger uten navnekollisjon -->
+  <xacro:macro name="qube" params="prefix">
+    <link name="${prefix}base_link"/>           <!-- usynlig referansepunkt -->
+    <link name="${prefix}stator_link">          <!-- svart boks -->
+      <visual>
+        <geometry>
+          <box size="${stator_size} ${stator_size} ${stator_size}"/>
+        </geometry>
+        <material name="black">
+          <color rgba="0 0 0 1"/>
+        </material>
+      </visual>
+    </link>
+    <link name="${prefix}rotor_link">           <!-- rød disk -->
+      <visual>
+        <geometry>
+          <cylinder length="${rotor_length}" radius="${rotor_radius}"/>
+        </geometry>
+        <material name="red">
+          <color rgba="1 0 0 1"/>
+        </material>
+      </visual>
+    </link>
+    <link name="${prefix}indicator_link">       <!-- hvit viser -->
+      <visual>
+        <geometry>
+          <box size="${indicator_length} ${indicator_width} ${indicator_width}"/>
+        </geometry>
+        <material name="white">
+          <color rgba="1 1 1 1"/>
+        </material>
+      </visual>
+    </link>
+    <!-- Boks plasseres oppå base_link -->
+    <joint name="${prefix}stator_joint" type="fixed">
+      <parent link="${prefix}base_link"/>
+      <child link="${prefix}stator_link"/>
+      <origin xyz="0 0 ${stator_size/2}" rpy="0 0 0"/>
+    </joint>
+    <!-- Roterende ledd - må hete motor_join -->
+    <joint name="${prefix}motor_joint" type="revolute">
+      <parent link="${prefix}stator_link"/>
+      <child link="${prefix}rotor_link"/>
+      <origin xyz="0 0 ${stator_size/2 + rotor_length/2}" rpy="0 0 0"/>
+      <axis xyz="0 0 1"/>
+      <limit lower="-3.1416" upper="3.1416" effort="1" velocity="1"/>
+    </joint>
+    <!-- Viseren montert på disken -->
+    <joint name="${prefix}indicator_joint" type="fixed">
+      <parent link="${prefix}rotor_link"/>
+      <child link="${prefix}indicator_link"/>
+      <origin xyz="${indicator_length/2} 0 ${rotor_length/2 + indicator_width/2}" rpy="0 0 0"/>
+    </joint>
+  </xacro:macro>
 </robot>

File: src/qube_description/urdf/qube.urdf.xacro (robot description, xacro)
@@ -1,58 +1,16 @@
 <?xml version="1.0"?>
-<robot xmlns:xacro="http://www.ros.org/wiki/xacro">
-  <xacro:property name="stator_size" value="0.102" />        <!-- boks (m) -->
-  <xacro:property name="rotor_radius" value="0.025" />       <!-- disk radius (m) -->
-  <xacro:property name="rotor_length" value="0.01" />        <!-- disk tykkelse (m) -->
-  <xacro:property name="indicator_length" value="0.025" />   <!-- viser lengde (m) -->
-  <xacro:property name="indicator_width" value="0.005" />    <!-- viser bredde (m) -->
-  <xacro:macro name="qube" params="prefix">     <!-- prefix unngår navnekollisjon -->
-    <link name="${prefix}base_link"/>           <!-- usynlig referansepunkt -->
-    <link name="${prefix}stator_link">          <!-- svart boks -->
-      <visual>
-        <geometry>
-          <box size="${stator_size} ${stator_size} ${stator_size}"/>
-        </geometry>
-        <material name="black">
-          <color rgba="0 0 0 1"/>
-        </material>
-      </visual>
-    </link>
-    <link name="${prefix}rotor_link">               <!-- rød disk -->
-      <visual>
-        <geometry>
-          <cylinder length="${rotor_length}" radius="${rotor_radius}"/>
-        </geometry>
-        <material name="red">
-          <color rgba="1 0 0 1"/>
-        </material>
-      </visual>
-    </link>
-    <link name="${prefix}indicator_link">           <!-- hvit viser -->
-      <visual>
-        <geometry>
-          <box size="${indicator_length} ${indicator_width} ${indicator_width}"/>
-        </geometry>
-        <material name="white">
-          <color rgba="1 1 1 1"/>
-        </material>
-      </visual>
-    </link>
-    <joint name="${prefix}stator_joint" type="fixed">           <!-- boks over referansepunkt -->
-      <parent link="${prefix}base_link"/>
-      <child link="${prefix}stator_link"/>
-      <origin xyz="0 0 ${stator_size/2}" rpy="0 0 0"/>
-    </joint>
-    <joint name="${prefix}motor_joint" type="revolute">         <!-- må hete motor_joint -->
-      <parent link="${prefix}stator_link"/>
-      <child link="${prefix}rotor_link"/>
-      <origin xyz="0 0 ${stator_size/2 + rotor_length/2}" rpy="0 0 0"/>
-      <axis xyz="0 0 1"/>
-      <limit lower="-3.1416" upper="3.1416" effort="1" velocity="1"/>
-    </joint>
-    <joint name="${prefix}indicator_joint" type="fixed">        <!-- en viser festet til disken -->
-      <parent link="${prefix}rotor_link"/>
-      <child link="${prefix}indicator_link"/>
-      <origin xyz="${indicator_length/2} 0 ${rotor_length/2 + indicator_width/2}" rpy="0 0 0"/>
-    </joint>
-  </xacro:macro>
+<!-- Enkel scene som plasserer én QUBE i origo. Brukes til visualisering i RViz. -->
+<robot xmlns:xacro="http://www.ros.org/wiki/xacro" name="qube">
+  <!-- Henter inn makroen fra makrofilen -->
+  <xacro:include filename="$(find qube_description)/urdf/qube.macro.xacro"/>
+  <!-- World-link er et fast referansepunkt i verdensrommet -->
+  <link name="world"/>
+  <!-- Kaller makroen med tomt prefix siden vi bare har én QUBE -->
+  <xacro:qube prefix=""/>
+  <!-- Fester QUBE-en til world i origo -->
+  <joint name="world_joint" type="fixed">
+    <parent link="world"/>
+    <child link="base_link"/>
+    <origin xyz="0 0 0" rpy="0 0 0"/>
+  </joint>
 </robot>
