Commit message: Inkluderer qube.urdf.xacro

File: install/qube_bringup/share/qube_bringup/urdf/controlled_qube.urdf.xacro (robot description, xacro)
@@ -1,69 +1,4 @@
 <?xml version="1.0"?>
 <robot xmlns:xacro="http://www.ros.org/wiki/xacro">
+  <xacro:include filename="$(find qube_description)/urdf/qube.urdf.xacro"/>
   <xacro:include filename="$(find qube_driver)/ros2_control/qube_driver.ros2_control.xacro"/>
-  <xacro:property name="stator_size" value="0.102" />        <!-- boks (m) -->
-  <xacro:property name="rotor_radius" value="0.025" />       <!-- disk radius (m) -->
-  <xacro:property name="rotor_length" value="0.01" />        <!-- disk tykkelse (m) -->
-  <xacro:property name="indicator_length" value="0.025" />   <!-- viser lengde (m) -->
-  <xacro:property name="indicator_width" value="0.005" />    <!-- viser bredde (m) -->
-  <xacro:macro name="qube" params="prefix">     <!-- prefix unngår navnekollisjon -->
-    <link name="${prefix}base_link"/>           <!-- usynlig referansepunkt -->
-    <link name="${prefix}stator_link">          <!-- svart boks -->
-      <visual>
-        <geometry>
-          <box size="${stator_size} ${stator_size} ${stator_size}"/>
-        </geometry>
-        <material name="black">
-          <color rgba="0 0 0 1"/>
-        </material>
-      </visual>
-    </link>
-    <link name="${prefix}rotor_link">               <!-- rød disk -->
-      <visual>
-        <geometry>
-          <cylinder length="${rotor_length}" radius="${rotor_radius}"/>
-        </geometry>
-        <material name="red">
-          <color rgba="1 0 0 1"/>
-        </material>
-      </visual>
-    </link>
-    <link name="${prefix}indicator_link">           <!-- hvit viser -->
-      <visual>
-        <geometry>
-          <box size="${indicator_length} ${indicator_width} ${indicator_width}"/>
-        </geometry>
-        <material name="white">
-          <color rgba="1 1 1 1"/>
-        </material>
-      </visual>
-    </link>
-    <joint name="${prefix}stator_joint" type="fixed">           <!-- boks over referansepunkt -->
-      <parent link="${prefix}base_link"/>
-      <child link="${prefix}stator_link"/>
-      <origin xyz="0 0 ${stator_size/2}" rpy="0 0 0"/>
-    </joint>
-    <joint name="${prefix}motor_joint" type="revolute">         <!-- må hete motor_joint -->
-      <parent link="${prefix}stator_link"/>
-      <child link="${prefix}rotor_link"/>
-      <origin xyz="0 0 ${stator_size/2 + rotor_length/2}" rpy="0 0 0"/>
-      <axis xyz="0 0 1"/>
-      <limit lower="-3.1416" upper="3.1416" effort="1" velocity="1"/>
-    </joint>
-    <joint name="${prefix}indicator_joint" type="fixed">        <!-- en viser festet til disken -->
-      <parent link="${prefix}rotor_link"/>
-      <child link="${prefix}indicator_link"/>
-      <origin xyz="${indicator_length/2} 0 ${rotor_length/2 + indicator_width/2}" rpy="0 0 0"/>
-    </joint>
-  </xacro:macro>
-  <xacro:arg name="baud_rate"  default="115200"/>
-  <xacro:arg name="device"     default="/dev/ttyUSB0"/>
-  <xacro:arg name="simulation" default="false"/>
-  <xacro:qube prefix=""/>
-  <xacro:qube_driver_ros2_control
-    name="qube_driver"
-    prefix=""
-    baud_rate="$(arg baud_rate)"
-    device="$(arg device)"
-    simulation="$(arg simulation)"/>
-</robot>
