Commit message: Lagt til kommentarer

File: src/qube_bringup/urdf/controlled_qube.urdf.xacro (robot description, xacro)
@@ -1,9 +1,12 @@
 <?xml version="1.0"?>
 <robot xmlns:xacro="http://www.ros.org/wiki/xacro" name="controlled_qube">
+  <!-- Henter inn scene-filen fra qube_description og ros2_control-grensesnittet til qube_driver -->
   <xacro:include filename="$(find qube_description)/urdf/qube.urdf.xacro"/>
   <xacro:include filename="$(find qube_driver)/ros2_control/qube_driver.ros2_control.xacro"/>
+  <!-- Default values; overskrives av argumentene fra bringup.launch.py -->
   <xacro:arg name="baud_rate"  default="115200"/>
   <xacro:arg name="device"     default="/dev/ttyACM0"/>
   <xacro:arg name="simulation" default="false"/>
+  <!-- Kaller qube_driver_ros2_control-makroen med argumentene over -->
   <xacro:qube_driver_ros2_control
     name="qube_driver"

File: src/qube_description/urdf/qube.macro.xacro (robot description, xacro)
@@ -40,5 +40,5 @@
       </visual>
     </link>
-    <!-- Boks plasseres oppå base_link -->
+    <!-- Boks plasseres på base_link -->
     <joint name="${prefix}stator_joint" type="fixed">
       <parent link="${prefix}base_link"/>
@@ -46,5 +46,5 @@
       <origin xyz="0 0 ${stator_size/2}" rpy="0 0 0"/>
     </joint>
-    <!-- Roterende ledd - må hete motor_join -->
+    <!-- Roterende ledd, må hete motor_joint -->
     <joint name="${prefix}motor_joint" type="revolute">
       <parent link="${prefix}stator_link"/>
@@ -52,5 +52,5 @@
       <origin xyz="0 0 ${stator_size/2 + rotor_length/2}" rpy="0 0 0"/>
       <axis xyz="0 0 1"/>
-      <limit lower="-3.1416" upper="3.1416" effort="1" velocity="1"/>
+      <limit lower="-3.1416" upper="3.1416" effort="1" velocity="1"/>  <!-- +- pi radianer -->
     </joint>
     <!-- Viseren montert på disken -->

File: src/qube_description/urdf/qube.urdf.xacro (robot description, xacro)
@@ -4,5 +4,5 @@
   <!-- Henter inn makroen fra makrofilen -->
   <xacro:include filename="$(find qube_description)/urdf/qube.macro.xacro"/>
-  <!-- World-link er et fast referansepunkt i verdensrommet -->
+  <!-- nullpunkt som alt annet er relativt til -->
   <link name="world"/>
   <!-- Kaller makroen med tomt prefix siden vi bare har én QUBE -->
